Commit message: pre ddsm-integration

File: src/robot_description/robot.urdf (robot description, URDF)
Before this commit: robot robot_description, 16 links, 15 joints
Joints:
- joint BLSteer: type revolute -> continuous
- joint BRSteer: type revolute -> continuous
- joint FLSteer: type revolute -> continuous
- joint FRSteer: type revolute -> continuous
